File: Hardware/SparkFun_GPS_ZED-F9K.sch (EAGLE design)
At the start: 74 parts, among them J3 QWIIC_RIGHT_ANGLE, J4 QWIIC_RIGHT_ANGLE, U1 DUAL-OPTO_HCPL-073LSOIC-8, U2 U-BLOX_ZED_F9K, U3 UHS_INVERTER_SCHMITT_TRIGGERS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, U4 UHS_INVERTER_SCHMITT_TRIGGERS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, U5 3.3V

Commit message: Changes name of I2C jumper to I2C, it was previously JP6
Parts:
- renumbered JP6 to I2C
Other:
- note added: "USB-C and Voltage Regulation: AP2112K"
- note removed: "Power"
Changed lines of the file:
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@@
 <part name="R23" library="SparkFun-Resistors" deviceset="4.7KOHM" device="-0402T-1/16W-1%" value="4.7k"/>
 <part name="R16" library="SparkFun-Resistors" deviceset="4.7KOHM" device="-0402T-1/16W-1%" value="4.7k"/>
-<part name="JP6" library="SparkFun-Jumpers" deviceset="JUMPER-SMT_3_2-NC_TRACE" device="_SILK" package3d_urn="urn:adsk.eagle:package:39289/1"/>
+<part name="I2C" library="SparkFun-Jumpers" deviceset="JUMPER-SMT_3_2-NC_TRACE" device="_SILK" package3d_urn="urn:adsk.eagle:package:39289/1"/>
 <part name="GND12" library="SparkFun-PowerSymbols" deviceset="GND" device=""/>
 <part name="SUPPLY5" library="SparkFun-PowerSymbols" deviceset="3.3V" device=""/>
@@
 <text x="421.64" y="7.62" size="2.54" layer="94" font="vector">v10</text>
 <text x="349.25" y="11.43" size="2.54" layer="94" font="vector">Elias Santistevan</text>
-<text x="86.36" y="269.24" size="3.81" layer="94" font="vector" align="center">GNSS/Dead Reckoning Module - ublox ZED-F9K</text>
-<text x="385.572" y="272.034" size="3.81" layer="94" font="vector" align="center">Battery</text>
-<text x="355.6" y="127" size="3.81" layer="94" font="vector" align="center">Connectors</text>
-<text x="248.92" y="127" size="3.81" layer="94" font="vector" align="center">Jumpers</text>
+<text x="86.36" y="269.24" size="2.54" layer="94" font="vector" align="center">GNSS/Dead Reckoning Module - ublox ZED-F9K</text>
+<text x="385.572" y="272.034" size="2.54" layer="94" font="vector" align="center">Battery</text>
+<text x="355.6" y="127" size="2.54" layer="94" font="vector" align="center">Connectors</text>
+<text x="248.92" y="127" size="2.54" layer="94" font="vector" align="center">Jumpers</text>
 <text x="228.6" y="76.2" size="2.54" layer="97" font="vector">Close Jumper for SPI</text>
 <text x="228.6" y="109.22" size="2.54" layer="97" font="vector">I2C Pull ups</text>
 <text x="218.186" y="54.102" size="2.54" layer="97" font="vector">Cut trace to disconnect respective LED</text>
-<text x="177.8" y="127" size="3.81" layer="94" font="vector" align="center">Antenna</text>
+<text x="177.8" y="127" size="2.54" layer="94" font="vector" align="center">Antenna</text>
 <wire x1="175.26" y1="134.62" x2="175.26" y2="279.4" width="0.1524" layer="97" style="shortdash"/>
 <wire x1="175.26" y1="134.62" x2="210.82" y2="134.62" width="0.1524" layer="97" style="shortdash"/>
@@
 <text x="304.8" y="236.22" size="1.27" layer="97" font="vector">VIN Range: 2.5V - 6V
 Max Current: 600mA</text>
-<text x="256.54" y="269.24" size="3.81" layer="94" font="vector" align="center">Power</text>
+<text x="256.54" y="269.24" size="2.54" layer="94" font="vector" align="center">USB-C and Voltage Regulation: AP2112K</text>
 <wire x1="210.82" y1="134.62" x2="292.1" y2="134.62" width="0.1524" layer="97" style="shortdash"/>
 <wire x1="292.1" y1="134.62" x2="340.36" y2="134.62" width="0.1524" layer="97" style="shortdash"/>
@@
 <wire x1="144.78" y1="134.62" x2="144.78" y2="0" width="0.2032" layer="97" style="shortdash"/>
 <wire x1="144.78" y1="134.62" x2="0" y2="134.62" width="0.2032" layer="97" style="shortdash"/>
-<text x="68.58" y="127" size="3.81" layer="94" font="vector" align="center">Wheel Tick and Direction Signal</text>
+<text x="68.58" y="127" size="2.54" layer="94" font="vector" align="center">Wheel Tick and Direction Signal</text>
 <text x="5.08" y="38.1" size="1.778" layer="97" font="vector">Wheel Tick/Direction
 Input: 3-24V</text>
@@
 <attribute name="VALUE" x="245.364" y="99.06" size="1.778" layer="96" font="vector" rot="R90" align="top-center"/>
 </instance>
-<instance part="JP6" gate="G$1" x="251.46" y="106.68" smashed="yes" rot="R270">
+<instance part="I2C" gate="G$1" x="251.46" y="106.68" smashed="yes" rot="R270">
 <attribute name="NAME" x="248.92" y="101.981" size="1.778" layer="95" font="vector"/>
 </instance>
@@
 </instance>
 <instance part="D2" gate="G$1" x="43.18" y="22.86" smashed="yes" rot="R90">
-<attribute name="NAME" x="47.498" y="26.162" size="1.778" layer="95" font="vector" rot="R180"/>
+<attribute name="NAME" x="47.498" y="25.4" size="1.778" layer="95" font="vector" rot="R180"/>
+<attribute name="VALUE" x="49.022" y="19.304" size="1.778" layer="96" font="vector" rot="R180" align="top-left"/>
 </instance>
 <instance part="R7" gate="G$1" x="68.326" y="106.426" smashed="yes" rot="R90">
@@
 </instance>
 <instance part="D1" gate="G$1" x="43.18" y="45.72" smashed="yes" rot="R90">
-<attribute name="NAME" x="47.498" y="49.022" size="1.778" layer="95" font="vector" rot="R180"/>
+<attribute name="NAME" x="47.752" y="49.276" size="1.778" layer="95" font="vector" rot="R180"/>
+<attribute name="VALUE" x="48.514" y="42.164" size="1.778" layer="96" font="vector" rot="R180" align="top-left"/>
 </instance>
 <instance part="SUPPLY23" gate="G$1" x="68.326" y="114.3" smashed="yes">
@@
 <instance part="U3" gate="U1" x="106.68" y="66.04" smashed="yes">
 <attribute name="NAME" x="96.52" y="74.422" size="1.778" layer="95"/>
-<attribute name="VALUE" x="96.52" y="55.88" size="1.778" layer="95"/>
+<attribute name="VALUE" x="91.44" y="55.88" size="1.778" layer="95"/>
 </instance>
 <instance part="U4" gate="U1" x="106.68" y="43.18" smashed="yes">
 <attribute name="NAME" x="96.52" y="51.562" size="1.778" layer="95"/>
-<attribute name="VALUE" x="96.52" y="33.02" size="1.778" layer="95"/>
+<attribute name="VALUE" x="91.44" y="33.02" size="1.778" layer="95"/>
 </instance>
 <instance part="TP1" gate="G$1" x="391.16" y="208.28" smashed="yes">
@@
 <net name="3.3V" class="0">
 <segment>
-<pinref part="JP6" gate="G$1" pin="2"/>
+<pinref part="I2C" gate="G$1" pin="2"/>
 <pinref part="SUPPLY5" gate="G$1" pin="3.3V"/>
 <wire x1="251.46" y1="111.76" x2="251.46" y2="114.3" width="0.1524" layer="91"/>
@@
 <pinref part="R23" gate="G$1" pin="2"/>
 <wire x1="259.08" y1="101.6" x2="259.08" y2="106.68" width="0.1524" layer="91"/>
-<pinref part="JP6" gate="G$1" pin="1"/>
+<pinref part="I2C" gate="G$1" pin="1"/>
 <wire x1="259.08" y1="106.68" x2="256.54" y2="106.68" width="0.1524" layer="91"/>
 </segment>
@@
 <net name="N$3" class="0">
 <segment>
-<pinref part="JP6" gate="G$1" pin="3"/>
+<pinref part="I2C" gate="G$1" pin="3"/>
 <wire x1="246.38" y1="106.68" x2="243.84" y2="106.68" width="0.1524" layer="91"/>
 <wire x1="243.84" y1="106.68" x2="243.84" y2="104.14" width="0.1524" layer="91"/>
