File: Hardware/SparkFun_GPS_ZED-F9K.sch (EAGLE design)
At the start: 74 parts, among them J3 QWIIC_RIGHT_ANGLE, J4 QWIIC_RIGHT_ANGLE, U1 DUAL-OPTO_HCPL-073LSOIC-8, U2 U-BLOX_ZED_F9K, U3 UHS_INVERTER_SCHMITT_TRIGGERS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, U4 UHS_INVERTER_SCHMITT_TRIGGERS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, U5 3.3V

Commit message: Adds PROD-ID to optoisolator
Parts:
- D9: value PESD0402 -> PESD0402-0402; device SparkFun-DiscreteSemi:PESD0402 -> SparkFun-DiscreteSemi:PESD0402-0402
Changed lines of the file:
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@@
 <part name="R10" library="SparkFun-Resistors" deviceset="33OHM_RA" device="-1206-1/16W-5%" value="33"/>
 <part name="R11" library="SparkFun-Resistors" deviceset="33OHM_RA" device="-1206-1/16W-5%" value="33"/>
-<part name="D9" library="SparkFun-DiscreteSemi" deviceset="PESD0402" device=""/>
+<part name="D9" library="SparkFun-DiscreteSemi" deviceset="PESD0402" device="-0402"/>
 <part name="E1" library="SparkFun-RF" deviceset="ANTENNA-SMA-GROUNDED" device="EDGE_SMA"/>
 <part name="U3" library="SparkFun-IC-Amplifiers" deviceset="UHS_INVERTER_SCHMITT_TRIGGER" device="SIP6" value="UHS_INVERTER_SCHMITT_TRIGGERSIP6"/>
@@
 <attribute name="VALUE" x="123.444" y="202.692" size="1.778" layer="96" font="vector" align="top-center"/>
 </instance>
-<instance part="D9" gate="G$1" x="180.34" y="75.438" smashed="yes" rot="R90">
+<instance part="D9" gate="D1" x="180.34" y="75.438" smashed="yes" rot="R90">
 <attribute name="NAME" x="176.784" y="77.978" size="1.778" layer="95" font="vector" rot="R270"/>
 <attribute name="VALUE" x="182.118" y="70.866" size="1.778" layer="96" font="vector" rot="R90" align="top-left"/>
@@
 <segment>
 <pinref part="GND4" gate="1" pin="GND"/>
-<pinref part="D9" gate="G$1" pin="1"/>
+<pinref part="D9" gate="D1" pin="1"/>
 <wire x1="172.72" y1="71.12" x2="172.72" y2="55.88" width="0.1524" layer="91"/>
 <wire x1="180.34" y1="72.898" x2="180.34" y2="71.12" width="0.1524" layer="91"/>
@@
 <junction x="185.42" y="83.82"/>
 <pinref part="FB1" gate="G$1" pin="1"/>
-<pinref part="D9" gate="G$1" pin="2"/>
+<pinref part="D9" gate="D1" pin="2"/>
 <wire x1="180.34" y1="80.518" x2="180.34" y2="83.82" width="0.1524" layer="91"/>
 <junction x="180.34" y="83.82"/>
