File: Hardware/SparkFun_GPS_ZED-F9K.brd (EAGLE design)
At the start: 43.2 x 50.8 mm, 149 parts, among them J3 QWIIC_RIGHT_ANGLE, J4 QWIIC_RIGHT_ANGLE, U1 DUAL-OPTO_HCPL-073LSOIC-8, U2 U-BLOX_ZED_F9K, U3 UHS_INVERTER_SCHMITT_TRIGGERS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, U4 UHS_INVERTER_SCHMITT_TRIGGERS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, U5 3.3V

Commit message: Fixes TXO/COPI silk to read TXO/CIPO
Parts:
- removed U$29: (no value), silkbot:#TXO#COPI#9
- added U$74: (no value), silkbot:#TXO#CIPO#9
Changed lines of the file:
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@@
 <element name="U$27" library="silkbot" package="#SDA##CS##10" value="" x="37.81" y="29.18" smashed="yes" rot="MR0"/>
 <element name="U$28" library="silkbot" package="#RXI#COPI#8" value="" x="37.3" y="26.69" smashed="yes" rot="MR0"/>
-<element name="U$29" library="silkbot" package="#TXO#COPI#9" value="" x="36.88" y="24.08" smashed="yes" rot="MR0"/>
 <element name="U$30" library="silkbot" package="#SCL#SCK#12" value="" x="37.6" y="21.56" smashed="yes" rot="MR0"/>
 <element name="U$31" library="silkbot" package="#D##6" value="" x="39.82" y="16.46" smashed="yes" rot="MR0"/>
@@
 <element name="TP1" library="SparkFun-Connectors" package="PAD.03X.05" value="TEST-POINT3X5" x="29.21" y="43.18" smashed="yes" rot="MR0"/>
 <element name="U$71" library="silk" package="#PPS#20" value="" x="3.81" y="16.383" smashed="yes"/>
+<element name="U$74" library="silkbot" package="#TXO#CIPO#9" value="" x="36.957" y="24.13" smashed="yes" rot="MR0"/>
 </elements>
 <signals>

Commit message: Adds PROD-ID to optoisolator
Parts:
- D9: value PESD0402 -> PESD0402-0402
Changed lines of the file:
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@@
 <element name="U1" library="SparkFun-DiscreteSemi" package="SO08" value="DUAL-OPTO_HCPL-073LSOIC-8" x="29.9426" y="9.2562" smashed="yes" rot="R90">
 <attribute name="NAME" x="26.59326875" y="5.4512" size="1.778" layer="25" rot="R90"/>
+<attribute name="PROD_ID" value="IC-15070" x="29.9426" y="9.2562" size="1.778" layer="27" rot="R90" display="off"/>
 <attribute name="VALUE" x="34.43493125" y="5.4512" size="1.778" layer="27" rot="R90"/>
 </element>
@@
 <element name="U$57" library="Orientation" package="Z0" value="" x="11.176" y="13.462" smashed="yes" rot="MR0"/>
 <element name="U$63" library="Orientation" package="Z0" value="" x="10.892" y="12.372" smashed="yes"/>
-<element name="D9" library="SparkFun-DiscreteSemi" package="0402" value="PESD0402" x="17.78" y="11.43" smashed="yes" rot="R180">
+<element name="D9" library="SparkFun-DiscreteSemi" package="0402" value="PESD0402-0402" x="17.78" y="11.43" smashed="yes" rot="R180">
 <attribute name="DIGIKEY_PART" value="PESD0402-140CT-ND" x="17.78" y="11.43" size="1.778" layer="27" rot="R180" display="off"/>
 <attribute name="MOUSE_PART" value="650-PESD0402-140" x="17.78" y="11.43" size="1.778" layer="27" rot="R180" display="off"/>
