File: Production/SparkFun_GPS_ZED-F9K-Panel.brd (EAGLE design)
At the start: 106 x 185.9 mm, 894 parts, among them J1 QWIIC_RIGHT_ANGLE, J10 QWIIC_RIGHT_ANGLE, J13 QWIIC_RIGHT_ANGLE, J16 QWIIC_RIGHT_ANGLE, J19 QWIIC_RIGHT_ANGLE, J22 QWIIC_RIGHT_ANGLE, J25 QWIIC_RIGHT_ANGLE, J28 QWIIC_RIGHT_ANGLE, J3 QWIIC_RIGHT_ANGLE, J31 QWIIC_RIGHT_ANGLE, J34 QWIIC_RIGHT_ANGLE, J4 QWIIC_RIGHT_ANGLE, U1 DUAL-OPTO_HCPL-073LSOIC-8, U10 UHS_INVERTER_SCHMITT_TRIGGERS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, U11 3.3V, U12 U-BLOX_ZED_F9K, U13 DUAL-OPTO_HCPL-073LSOIC-8, U14 UHS_INVERTER_SCHMITT_TRIGGERS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, U15 UHS_INVERTER_SCHMITT_TRIGGERS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, U16 3.3V, U17 U-BLOX_ZED_F9K, U18 DUAL-OPTO_HCPL-073LSOIC-8, U19 UHS_INVERTER_SCHMITT_TRIGGERS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, U2 U-BLOX_ZED_F9K, U20 UHS_INVERTER_SCHMITT_TRIGGERS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, U21 3.3V, U22 U-BLOX_ZED_F9K, U23 DUAL-OPTO_HCPL-073LSOIC-8, U24 UHS_INVERTER_SCHMITT_TRIGGERS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, U25 UHS_INVERTER_SCHMITT_TRIGGERS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, U26 3.3V, U27 U-BLOX_ZED_F9K, U28 DUAL-OPTO_HCPL-073LSOIC-8, U29 UHS_INVERTER_SCHMITT_TRIGGERS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, U3 UHS_INVERTER_SCHMITT_TRIGGERS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, U30 UHS_INVERTER_SCHMITT_TRIGGERS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, U4 UHS_INVERTER_SCHMITT_TRIGGERS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, U5 3.3V, U6 3.3V, U7 U-BLOX_ZED_F9K, U8 DUAL-OPTO_HCPL-073LSOIC-8, U9 UHS_INVERTER_SCHMITT_TRIGGERS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

Commit message: Panel
Parts:
- U$115, U$188, U$261, U$334, U$407: device silkbot:#TXO#COPI#9 -> silkbot:#SCL#SCK#12
- U$116, U$189, U$262, U$335, U$408: device silkbot:#SCL#SCK#12 -> silkbot:#D##6
- U$117, U$190, U$263, U$336, U$409: device silkbot:#D##6 -> silkbot:#D##7
- U$118, U$191, U$264, U$337, U$410: device silkbot:#D##7 -> silkbot:#W##4
- U$119, U$192, U$265, U$338, U$411: device silkbot:#W##4 -> silkbot:#W##5
- U$120, U$193, U$266, U$339, U$412: device silkbot:#W##5 -> silk:#GND#0
- U$121, U$194, U$267, U$340, U$413: device silk:#GND#0 -> silk:#3V3#6
- U$122, U$195, U$268, U$341, U$414: device silk:#3V3#6 -> silk:#SDA#6
- U$123, U$196, U$269, U$342, U$415: device silk:#SDA#6 -> silk:#SCL#7
- U$124, U$197, U$270, U$343, U$416: device silk:#SCL#7 -> silkbot:#TXR#3
- U$125, U$198, U$271, U$344, U$417: device silkbot:#TXR#3 -> silkbot:##RST##16
- U$126, U$199, U$272, U$345, U$418: device silkbot:##RST##16 -> silkbot:##SFBT##17
- U$127, U$200, U$273, U$346, U$419: device silkbot:##SFBT##17 -> silk:#INT#8
- U$128, U$201, U$274, U$347, U$420: device silk:#INT#8 -> silkbot:#PPS#0
- U$129, U$202, U$275, U$348, U$421: device silkbot:#PPS#0 -> silk:#RTK#25
- U$130, U$203, U$276, U$349, U$422: device silk:#RTK#25 -> silk:#GEO#24
- U$131, U$204, U$277, U$350, U$423: device silk:#GEO#24 -> silk:#PPS#21
- U$132, U$205, U$278, U$351, U$424: device silk:#PPS#21 -> silk:#PWR#23
- U$133, U$206, U$279, U$352, U$425: device silk:#PWR#23 -> silk:#SPI#22
- U$134, U$207, U$280, U$353, U$426: device silk:#SPI#22 -> silk:#I2C#23
- U$135, U$208, U$281, U$354, U$427: device silk:#I2C#23 -> silk:#RXI2#227
- U$136, U$209, U$282, U$355, U$428: device silk:#RXI2#227 -> silkbot:#TXO2#1
- U$137, U$210, U$283, U$356, U$429: device silkbot:#TXO2#1 -> silk:#GND#0
- U$138, U$211, U$284, U$357, U$430: device silk:#GND#0 -> silk:BLK227
- U$139, U$212, U$285, U$358, U$431: device silk:BLK227 -> silk:GRN228
- U$140, U$213, U$286, U$359, U$432: device silk:GRN228 -> silk:GNSS#DEAD_RECKONING230
- U$141, U$214, U$287, U$360, U$433: device silk:GNSS#DEAD_RECKONING230 -> silk:ZED#F9K230
- U$142, U$215, U$288, U$361, U$434: device silk:ZED#F9K230 -> silk:L1#L2229
- U$143, U$216, U$289, U$362, U$435: device silk:L1#L2229 -> silk:ANTENNA229
- U$144, U$217, U$290, U$363, U$436: device silk:ANTENNA229 -> silk:ZED#F9K230
- U$145, U$218, U$291, U$364, U$437: device silk:ZED#F9K230 -> silk:#PPS#20
- U$146, U$219, U$292, U$365, U$438: device silk:#PPS#20 -> silkbot:#TXO#CIPO#9
- U$29: device silkbot:#TXO#COPI#9 -> Dead#Reckoning#GPS#board#silk#FINAL#png:DEAD#RECKONING#GPS#BOARD#SILK#FINAL#JPG
- U$74: device Dead#Reckoning#GPS#board#silk#FINAL#png:DEAD#RECKONING#GPS#BOARD#SILK#FINAL#JPG -> silkbot:#TXO#CIPO#9
- moved U$193 42.4 mm to (3.97, 92.7)
- moved U$266 42.4 mm to (47.7, 92.7)
- moved U$120 42.4 mm to (47.7, 36.8)
- moved U$339 42.4 mm to (3.97, 148.5)
- moved U$412 42.4 mm to (47.7, 148.5)
- moved U$359 41.0 mm to (22.1, 122.8)
- moved U$432 41.0 mm to (65.8, 122.8)
- moved U$140 41.0 mm to (65.8, 11.1)
- moved U$213 41.0 mm to (22.1, 66.9)
- moved U$286 41.0 mm to (65.8, 66.9)
- moved U$129 34.8 mm to (79.7, 3.17)
- moved U$275 34.8 mm to (79.7, 59.0)
- moved U$202 34.8 mm to (36.0, 59.0)
- moved U$421 34.8 mm to (79.7, 114.9)
- moved U$348 34.8 mm to (36.0, 114.9)
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